Commit message: w

File: leg/Walker_description/urdf/Walker.xacro (robot description, xacro)
@@ -13,5 +13,5 @@
     <origin xyz="0 0 0" rpy="0 0 0"/>
     <geometry>
-      <mesh filename="leg/Walker_description/meshes/base_link.stl" scale="0.001 0.001 0.001"/>
+      <mesh filename="package://Walker_description/meshes/base_link.stl" scale="0.001 0.001 0.001"/>
     </geometry>
     <material name="silver"/>
@@ -20,5 +20,5 @@
     <origin xyz="0 0 0" rpy="0 0 0"/>
     <geometry>
-      <mesh filename="leg/Walker_description/meshes/base_link.stl" scale="0.001 0.001 0.001"/>
+      <mesh filename="package://Walker_description/meshes/base_link.stl" scale="0.001 0.001 0.001"/>
     </geometry>
   </collision>
@@ -33,5 +33,5 @@
     <origin xyz="-0.0 -0.015 0.03" rpy="0 0 0"/>
     <geometry>
-      <mesh filename="leg/Walker_description/meshes/thigh_1.stl" scale="0.001 0.001 0.001"/>
+      <mesh filename="package://Walker_description/meshes/thigh_1.stl" scale="0.001 0.001 0.001"/>
     </geometry>
     <material name="silver"/>
@@ -40,5 +40,5 @@
     <origin xyz="-0.0 -0.015 0.03" rpy="0 0 0"/>
     <geometry>
-      <mesh filename="leg/Walker_description/meshes/thigh_1.stl" scale="0.001 0.001 0.001"/>
+      <mesh filename="package://Walker_description/meshes/thigh_1.stl" scale="0.001 0.001 0.001"/>
     </geometry>
   </collision>
@@ -53,5 +53,5 @@
     <origin xyz="-0.0 -0.015 0.11" rpy="0 0 0"/>
     <geometry>
-      <mesh filename="leg/Walker_description/meshes/knee_1.stl" scale="0.001 0.001 0.001"/>
+      <mesh filename="package://Walker_description/meshes/knee_1.stl" scale="0.001 0.001 0.001"/>
     </geometry>
     <material name="silver"/>
@@ -60,5 +60,5 @@
     <origin xyz="-0.0 -0.015 0.11" rpy="0 0 0"/>
     <geometry>
-      <mesh filename="leg/Walker_description/meshes/knee_1.stl" scale="0.001 0.001 0.001"/>
+      <mesh filename="package://Walker_description/meshes/knee_1.stl" scale="0.001 0.001 0.001"/>
     </geometry>
   </collision>
@@ -73,5 +73,5 @@
     <origin xyz="-0.0 -0.015 0.13" rpy="0 0 0"/>
     <geometry>
-      <mesh filename="leg/Walker_description/meshes/shin_1.stl" scale="0.001 0.001 0.001"/>
+      <mesh filename="package://Walker_description/meshes/shin_1.stl" scale="0.001 0.001 0.001"/>
     </geometry>
     <material name="silver"/>
@@ -80,5 +80,5 @@
     <origin xyz="-0.0 -0.015 0.13" rpy="0 0 0"/>
     <geometry>
-      <mesh filename="leg/Walker_description/meshes/shin_1.stl" scale="0.001 0.001 0.001"/>
+      <mesh filename="package://Walker_description/meshes/shin_1.stl" scale="0.001 0.001 0.001"/>
     </geometry>
   </collision>
@@ -93,5 +93,5 @@
     <origin xyz="-0.0 -0.015 0.21" rpy="0 0 0"/>
     <geometry>
-      <mesh filename="leg/Walker_description/meshes/ankle_1.stl" scale="0.001 0.001 0.001"/>
+      <mesh filename="package://Walker_description/meshes/ankle_1.stl" scale="0.001 0.001 0.001"/>
     </geometry>
     <material name="silver"/>
@@ -100,5 +100,5 @@
     <origin xyz="-0.0 -0.015 0.21" rpy="0 0 0"/>
     <geometry>
-      <mesh filename="leg/Walker_description/meshes/ankle_1.stl" scale="0.001 0.001 0.001"/>
+      <mesh filename="package://Walker_description/meshes/ankle_1.stl" scale="0.001 0.001 0.001"/>
     </geometry>
   </collision>
@@ -113,5 +113,5 @@
     <origin xyz="-0.015 0.0 0.23" rpy="0 0 0"/>
     <geometry>
-      <mesh filename="leg/Walker_description/meshes/ankle_roll_1.stl" scale="0.001 0.001 0.001"/>
+      <mesh filename="package://Walker_description/meshes/ankle_roll_1.stl" scale="0.001 0.001 0.001"/>
     </geometry>
     <material name="silver"/>
@@ -120,5 +120,5 @@
     <origin xyz="-0.015 0.0 0.23" rpy="0 0 0"/>
     <geometry>
-      <mesh filename="leg/Walker_description/meshes/ankle_roll_1.stl" scale="0.001 0.001 0.001"/>
+      <mesh filename="package://Walker_description/meshes/ankle_roll_1.stl" scale="0.001 0.001 0.001"/>
     </geometry>
   </collision>
@@ -133,5 +133,5 @@
     <origin xyz="-0.0 0.0 0.26" rpy="0 0 0"/>
     <geometry>
-      <mesh filename="leg/Walker_description/meshes/foot_1.stl" scale="0.001 0.001 0.001"/>
+      <mesh filename="package://Walker_description/meshes/foot_1.stl" scale="0.001 0.001 0.001"/>
     </geometry>
     <material name="silver"/>
@@ -140,5 +140,5 @@
     <origin xyz="-0.0 0.0 0.26" rpy="0 0 0"/>
     <geometry>
-      <mesh filename="leg/Walker_description/meshes/foot_1.stl" scale="0.001 0.001 0.001"/>
+      <mesh filename="package://Walker_description/meshes/foot_1.stl" scale="0.001 0.001 0.001"/>
     </geometry>
   </collision>
@@ -149,5 +149,4 @@
   <child link="thigh_1"/>
   <axis xyz="0.0 1.0 0.0"/>
-  <limit lower="-1.57" upper="1.57" effort="100" velocity="1.0"/>
 </joint>
 <joint name="knee_1" type="continuous">
@@ -156,5 +155,4 @@
   <child link="knee_1"/>
   <axis xyz="-0.0 1.0 -0.0"/>
-  <limit lower="-1.57" upper="1.57" effort="100" velocity="1.0"/>
 </joint>
 <joint name="knee_2" type="continuous">
@@ -163,5 +161,4 @@
   <child link="shin_1"/>
   <axis xyz="0.0 1.0 -0.0"/>
-  <limit lower="-1.57" upper="1.57" effort="100" velocity="1.0"/>
 </joint>
 <joint name="ankle" type="continuous">
@@ -170,5 +167,4 @@
   <child link="ankle_1"/>
   <axis xyz="0.0 1.0 -0.0"/>
-  <limit lower="-1.57" upper="1.57" effort="100" velocity="1.0"/>
 </joint>
 <joint name="Revolute 112" type="continuous">
@@ -177,5 +173,4 @@
   <child link="ankle_roll_1"/>
   <axis xyz="1.0 -0.0 0.0"/>
-  <limit lower="-1.57" upper="1.57" effort="100" velocity="1.0"/>
 </joint>
 <joint name="Rigid 113" type="fixed">
