Commit message: k

File: Walker.urdf (robot description, URDF)
Before this commit: robot Walker, 7 links, 6 joints
Links:
- removed link link_1_1
- removed link link_2_1
- removed link link_3_1
- removed link link_4_1
- removed link servo_1_1
- removed link servo_2_1
- added link end_effector_1, mass 0.03567910939661666; collision mesh filename=leg/Walker_description/meshes/end_effector_1.stl scale=0.001 0.001 0.001; visual mesh filename=leg/Walker_description/meshes/end_effector_1.stl scale=0.001 0.001 0.001
- added link right_ankle_1, mass 0.02207862348176061; collision mesh filename=leg/Walker_description/meshes/right_ankle_1.stl scale=0.001 0.001 0.001; visual mesh filename=leg/Walker_description/meshes/right_ankle_1.stl scale=0.001 0.001 0.001
- added link right_foot_1, mass 0.031643029734136574; collision mesh filename=leg/Walker_description/meshes/right_foot_1.stl scale=0.001 0.001 0.001; visual mesh filename=leg/Walker_description/meshes/right_foot_1.stl scale=0.001 0.001 0.001
- added link right_hip_1, mass 0.015518960743906235; collision mesh filename=leg/Walker_description/meshes/right_hip_1.stl scale=0.001 0.001 0.001; visual mesh filename=leg/Walker_description/meshes/right_hip_1.stl scale=0.001 0.001 0.001
- added link right_knee_1, mass 0.03724513708022543; collision mesh filename=leg/Walker_description/meshes/right_knee_1.stl scale=0.001 0.001 0.001; visual mesh filename=leg/Walker_description/meshes/right_knee_1.stl scale=0.001 0.001 0.001
- added link right_shin_1, mass 0.04838185238285193; collision mesh filename=leg/Walker_description/meshes/right_shin_1.stl scale=0.001 0.001 0.001; visual mesh filename=leg/Walker_description/meshes/right_shin_1.stl scale=0.001 0.001 0.001
- added link right_thigh_1, mass 0.04841117262972764; collision mesh filename=leg/Walker_description/meshes/right_thigh_1.stl scale=0.001 0.001 0.001; visual mesh filename=leg/Walker_description/meshes/right_thigh_1.stl scale=0.001 0.001 0.001
- link base_link: mass 0.025300892916588436 -> 0.027166123584619145
Joints:
- removed joint Revolute 41
- removed joint Revolute 42
- removed joint Revolute 44
- removed joint Revolute 45
- removed joint Rigid 40
- removed joint Rigid 43
- added joint Revolute 85: type continuous, parent base_link, child right_hip_1, origin xyz=0.018625 0.0 -0.037125 rpy=0 0 0, axis 1.0 0.0 -0.0
- added joint Revolute 86: type continuous, parent right_hip_1, child right_thigh_1, origin xyz=-0.018626 0.018625 -0.040607 rpy=0 0 0, axis 0.0 -1.0 -0.0
- added joint Revolute 87: type fixed, parent right_thigh_1, child right_knee_1, origin xyz=0.0 -0.00355 -0.065 rpy=0 0 0, axis 0.0 -1.0 -0.0
- added joint Revolute 88: type continuous, parent right_knee_1, child right_shin_1, origin xyz=0.0 0.00355 -0.030981 rpy=0 0 0, axis -0.0 1.0 0.0
- added joint Revolute 89: type continuous, parent right_shin_1, child right_ankle_1, origin xyz=0.0 -0.00355 -0.065 rpy=0 0 0, axis 0.0 -1.0 -0.0
- added joint Revolute 91: type continuous, parent right_ankle_1, child right_foot_1, origin xyz=0.018626 -0.002575 -0.040247 rpy=0 0 0, axis 1.0 0.0 0.0
- added joint Rigid 92: type fixed, parent right_foot_1, child end_effector_1, origin xyz=-0.018625 -0.0125 -0.020075 rpy=0 0 0

File: trash/Walker.urdf (robot description, URDF)
Before this commit: robot Walker, 4 links, 3 joints
Links:
- removed link link_1_1
- removed link link_2_1
- removed link link_3_1
- added link right_ankle_1, mass 0.02214685736623212; collision mesh filename=leg/Walker_description/meshes/right_ankle_1.stl scale=0.001 0.001 0.001; visual mesh filename=leg/Walker_description/meshes/right_ankle_1.stl scale=0.001 0.001 0.001
- added link right_foot_1, mass 0.02421909542027639; collision mesh filename=leg/Walker_description/meshes/right_foot_1.stl scale=0.001 0.001 0.001; visual mesh filename=leg/Walker_description/meshes/right_foot_1.stl scale=0.001 0.001 0.001
- added link right_hip_1, mass 0.0160262455466391; collision mesh filename=leg/Walker_description/meshes/right_hip_1.stl scale=0.001 0.001 0.001; visual mesh filename=leg/Walker_description/meshes/right_hip_1.stl scale=0.001 0.001 0.001
- added link right_knee_1, mass 0.037245137080226885; collision mesh filename=leg/Walker_description/meshes/right_knee_1.stl scale=0.001 0.001 0.001; visual mesh filename=leg/Walker_description/meshes/right_knee_1.stl scale=0.001 0.001 0.001
- added link right_shin_1, mass 0.02773184406480059; collision mesh filename=leg/Walker_description/meshes/right_shin_1.stl scale=0.001 0.001 0.001; visual mesh filename=leg/Walker_description/meshes/right_shin_1.stl scale=0.001 0.001 0.001
- added link right_thigh_1, mass 0.02773211376260182; collision mesh filename=leg/Walker_description/meshes/right_thigh_1.stl scale=0.001 0.001 0.001; visual mesh filename=leg/Walker_description/meshes/right_thigh_1.stl scale=0.001 0.001 0.001
- added link servo_1_1, mass 0.07169587899149946; collision mesh filename=leg/Walker_description/meshes/servo_1_1.stl scale=0.001 0.001 0.001; visual mesh filename=leg/Walker_description/meshes/servo_1_1.stl scale=0.001 0.001 0.001
- added link servo_2_1, mass 0.07170037534026219; collision mesh filename=leg/Walker_description/meshes/servo_2_1.stl scale=0.001 0.001 0.001; visual mesh filename=leg/Walker_description/meshes/servo_2_1.stl scale=0.001 0.001 0.001
- added link servo_3_1, mass 0.07170037538363631; collision mesh filename=leg/Walker_description/meshes/servo_3_1.stl scale=0.001 0.001 0.001; visual mesh filename=leg/Walker_description/meshes/servo_3_1.stl scale=0.001 0.001 0.001
- added link servo_4_1, mass 0.07169587899501298; collision mesh filename=leg/Walker_description/meshes/servo_4_1.stl scale=0.001 0.001 0.001; visual mesh filename=leg/Walker_description/meshes/servo_4_1.stl scale=0.001 0.001 0.001
- link base_link: mass 0.610458688268196 -> 0.0065722113345469; geometry collision mesh filename=leg/Walker_description/meshes/base_link.stl scale=0.001 0.001 0.001; visual mesh filename=leg/Walker_description/meshes/base_link.stl scale=0.001 0.001 0.001
Joints:
- removed joint Revolute 27
- removed joint Revolute 28
- removed joint Revolute 29
- added joint Revolute 59: type continuous, parent servo_1_1, child right_hip_1, origin xyz=0.0047 -0.01 -0.03275 rpy=0 0 0, axis 1.0 0.0 -0.0
- added joint Revolute 60: type continuous, parent right_hip_1, child servo_2_1, origin xyz=-0.018668 0.018621 -0.040607 rpy=0 0 0, axis 0.0 -1.0 1e-06
- added joint Revolute 64: type continuous, parent right_knee_1, child servo_3_1, origin xyz=0.0 0.00355 -0.030981 rpy=0 0 0, axis -0.0 1.0 -1e-06
- added joint Revolute 66: type continuous, parent right_shin_1, child right_ankle_1, origin xyz=0.01 0.00115 -0.03225 rpy=0 0 0, axis 0.0 -1.0 1e-06
- added joint Revolute 67: type continuous, parent right_ankle_1, child servo_4_1, origin xyz=0.018668 -0.002575 -0.040247 rpy=0 0 0, axis 1.0 0.0 -0.0
- added joint Rigid 58: type fixed, parent base_link, child servo_1_1, origin xyz=0.013925 0.009999 -0.004375 rpy=0 0 0
- added joint Rigid 61: type fixed, parent servo_2_1, child right_thigh_1, origin xyz=-0.01 -0.0047 -0.03275 rpy=0 0 0
- added joint Rigid 62: type fixed, parent right_thigh_1, child right_knee_1, origin xyz=0.01 0.00115 -0.03225 rpy=0 0 0
- added joint Rigid 65: type fixed, parent servo_3_1, child right_shin_1, origin xyz=-0.01 -0.0047 -0.03275 rpy=0 0 0
- added joint Rigid 68: type fixed, parent servo_4_1, child right_foot_1, origin xyz=-0.0047 -0.03275 0.01 rpy=0 0 0

Commit message: l

File: Walker.urdf (robot description, URDF)
Before this commit: robot Walker, 8 links, 7 joints
Links:
- removed link end_effector_1
- removed link right_ankle_1
- removed link right_foot_1
- removed link right_hip_1
- removed link right_knee_1
- removed link right_shin_1
- removed link right_thigh_1
- added link Component212_1, mass 0.7031706971853583; collision mesh filename=leg/Walker_description/meshes/Component212_1.stl scale=0.001 0.001 0.001; visual mesh filename=leg/Walker_description/meshes/Component212_1.stl scale=0.001 0.001 0.001
- added link Component214_1, mass 0.6358499999999999; collision mesh filename=leg/Walker_description/meshes/Component214_1.stl scale=0.001 0.001 0.001; visual mesh filename=leg/Walker_description/meshes/Component214_1.stl scale=0.001 0.001 0.001
- added link Component215_1, mass 0.7031706971853583; collision mesh filename=leg/Walker_description/meshes/Component215_1.stl scale=0.001 0.001 0.001; visual mesh filename=leg/Walker_description/meshes/Component215_1.stl scale=0.001 0.001 0.001
- added link Component218_1, mass 0.27927069718535813; collision mesh filename=leg/Walker_description/meshes/Component218_1.stl scale=0.001 0.001 0.001; visual mesh filename=leg/Walker_description/meshes/Component218_1.stl scale=0.001 0.001 0.001
- link base_link: mass 0.027166123584619145 -> 0.27927069718535813
Joints:
- removed joint Revolute 85
- removed joint Revolute 86
- removed joint Revolute 87
- removed joint Revolute 88
- removed joint Revolute 89
- removed joint Revolute 91
- removed joint Rigid 92
- added joint Revolute 102: type continuous, parent base_link, child Component212_1, origin xyz=0.0 -0.015 -0.03 rpy=0 0 0, axis 0.0 1.0 0.0
- added joint Revolute 103: type continuous, parent Component212_1, child Component215_1, origin xyz=0.0 0.0 -0.08 rpy=0 0 0, axis 0.0 1.0 0.0
- added joint Revolute 104: type continuous, parent Component215_1, child Component218_1, origin xyz=0.0 0.0 -0.08 rpy=0 0 0, axis 0.0 1.0 0.0
- added joint Rigid 105: type fixed, parent Component218_1, child Component214_1, origin xyz=0.0 0.015 -0.03 rpy=0 0 0

File: trash/Walker.urdf (robot description, URDF)
Before this commit: robot Walker, 11 links, 10 joints
Links:
- removed link servo_1_1
- removed link servo_2_1
- removed link servo_3_1
- removed link servo_4_1
- added link end_effector_1, mass 0.010298171671797838; collision mesh filename=leg/Walker_description/meshes/end_effector_1.stl scale=0.001 0.001 0.001; visual mesh filename=leg/Walker_description/meshes/end_effector_1.stl scale=0.001 0.001 0.001
- link base_link: mass 0.0065722113345469 -> 0.027166123584619145
- link right_ankle_1: mass 0.02214685736623212 -> 0.02207862348176061
- link right_foot_1: mass 0.02421909542027639 -> 0.031643029734136574
- link right_hip_1: mass 0.0160262455466391 -> 0.015518960743906235
- link right_knee_1: mass 0.037245137080226885 -> 0.03724513708022543
- link right_shin_1: mass 0.02773184406480059 -> 0.04838185238285193
- link right_thigh_1: mass 0.02773211376260182 -> 0.04841117262972764
Joints:
- removed joint Revolute 59
- removed joint Revolute 60
- removed joint Revolute 64
- removed joint Revolute 66
- removed joint Revolute 67
- removed joint Rigid 58
- removed joint Rigid 61
- removed joint Rigid 62
- removed joint Rigid 65
- removed joint Rigid 68
- added joint Revolute 85: type continuous, parent base_link, child right_hip_1, origin xyz=0.018625 0.0 -0.037125 rpy=0 0 0, axis 1.0 0.0 -0.0
- added joint Revolute 86: type continuous, parent right_hip_1, child right_thigh_1, origin xyz=-0.018626 0.018625 -0.040607 rpy=0 0 0, axis 0.0 -1.0 -0.0
- added joint Revolute 88: type continuous, parent right_knee_1, child right_shin_1, origin xyz=0.0 0.00355 -0.030981 rpy=0 0 0, axis -0.0 1.0 0.0
- added joint Revolute 89: type continuous, parent right_shin_1, child right_ankle_1, origin xyz=0.0 -0.00355 -0.065 rpy=0 0 0, axis 0.0 -1.0 -0.0
- added joint Revolute 91: type continuous, parent right_ankle_1, child right_foot_1, origin xyz=0.018626 -0.002575 -0.040247 rpy=0 0 0, axis 1.0 0.0 0.0
- added joint Rigid 87: type fixed, parent right_thigh_1, child right_knee_1, origin xyz=0.0 -0.00355 -0.065 rpy=0 0 0
- added joint Rigid 93: type fixed, parent right_foot_1, child end_effector_1, origin xyz=-0.018625 -0.0125 -0.020075 rpy=0 0 0

Commit message: m

File: Walker.urdf (robot description, URDF)
Before this commit: robot Walker, 5 links, 4 joints
Links:
- removed link Component214_1
Joints:
- removed joint Rigid 105

Commit message: n

File: Walker.urdf (robot description, URDF)
Before this commit: robot Walker, 4 links, 3 joints
Joints:
- joint Revolute 103: limit (none) -> lower=0 upper=3.14 effort=100 velocity=1.0; type continuous -> revolute

Commit message: o

File: Walker.urdf (robot description, URDF)
Before this commit: robot Walker, 4 links, 3 joints
Joints:
- joint Revolute 102: limit (none) -> lower=-3.14 upper=3.14 effort=100 velocity=1.0; type continuous -> revolute
- joint Revolute 103: limit lower=0 upper=3.14 effort=100 velocity=1.0 -> lower=-3.14 upper=3.14 effort=100 velocity=1.0
- joint Revolute 104: limit (none) -> lower=-3.14 upper=3.14 effort=100 velocity=1.0; type continuous -> revolute

Commit message: p

File: Walker.urdf (robot description, URDF)
Before this commit: robot Walker, 4 links, 3 joints
Links:
- removed link Component212_1
- removed link Component215_1
- removed link Component218_1
- added link ankle_1, mass 0.16126943544832453; collision mesh filename=leg/Untitled_description/meshes/ankle_1.stl scale=0.001 0.001 0.001; visual mesh filename=leg/Untitled_description/meshes/ankle_1.stl scale=0.001 0.001 0.001
- added link end_1, mass 0.2835812441560948; collision mesh filename=leg/Untitled_description/meshes/end_1.stl scale=0.001 0.001 0.001; visual mesh filename=leg/Untitled_description/meshes/end_1.stl scale=0.001 0.001 0.001
- added link foot_1, mass 0.07564259890689244; collision mesh filename=leg/Untitled_description/meshes/foot_1.stl scale=0.001 0.001 0.001; visual mesh filename=leg/Untitled_description/meshes/foot_1.stl scale=0.001 0.001 0.001
- added link hip_1, mass 0.16126943544832453; collision mesh filename=leg/Untitled_description/meshes/hip_1.stl scale=0.001 0.001 0.001; visual mesh filename=leg/Untitled_description/meshes/hip_1.stl scale=0.001 0.001 0.001
- added link knee_1, mass 0.3524642857407411; collision mesh filename=leg/Untitled_description/meshes/knee_1.stl scale=0.001 0.001 0.001; visual mesh filename=leg/Untitled_description/meshes/knee_1.stl scale=0.001 0.001 0.001
- added link servo1_1, mass 0.288363601261775; collision mesh filename=leg/Untitled_description/meshes/servo1_1.stl scale=0.001 0.001 0.001; visual mesh filename=leg/Untitled_description/meshes/servo1_1.stl scale=0.001 0.001 0.001
- added link servo_2_1, mass 0.2883636012617749; collision mesh filename=leg/Untitled_description/meshes/servo_2_1.stl scale=0.001 0.001 0.001; visual mesh filename=leg/Untitled_description/meshes/servo_2_1.stl scale=0.001 0.001 0.001
- added link servo_3_1, mass 0.2883636012617749; collision mesh filename=leg/Untitled_description/meshes/servo_3_1.stl scale=0.001 0.001 0.001; visual mesh filename=leg/Untitled_description/meshes/servo_3_1.stl scale=0.001 0.001 0.001
- added link servo_4_1, mass 0.28836360126173155; collision mesh filename=leg/Untitled_description/meshes/servo_4_1.stl scale=0.001 0.001 0.001; visual mesh filename=leg/Untitled_description/meshes/servo_4_1.stl scale=0.001 0.001 0.001
- added link shin_1, mass 0.3751668513433219; collision mesh filename=leg/Untitled_description/meshes/shin_1.stl scale=0.001 0.001 0.001; visual mesh filename=leg/Untitled_description/meshes/shin_1.stl scale=0.001 0.001 0.001
- added link thigh_1, mass 0.3751668513433219; collision mesh filename=leg/Untitled_description/meshes/thigh_1.stl scale=0.001 0.001 0.001; visual mesh filename=leg/Untitled_description/meshes/thigh_1.stl scale=0.001 0.001 0.001
- link base_link: mass 0.27927069718535813 -> 0.07564259890699374; geometry collision mesh filename=leg/Untitled_description/meshes/base_link.stl scale=0.001 0.001 0.001; visual mesh filename=leg/Untitled_description/meshes/base_link.stl scale=0.001 0.001 0.001
Joints:
- removed joint Revolute 102
- removed joint Revolute 103
- removed joint Revolute 104
- added joint Revolute 2: type revolute, parent servo1_1, child hip_1, origin xyz=0.01865 -0.0 -0.035 rpy=0 0 0, axis 1.0 -0.0 0.0, limit lower=-1.57 upper=1.57 effort=100 velocity=1.0
- added joint Revolute 3: type revolute, parent hip_1, child servo_2_1, origin xyz=-0.01865 -0.01865 -0.04 rpy=0 0 0, axis 0.0 1.0 -0.0, limit lower=-1.57 upper=1.57 effort=100 velocity=1.0
- added joint Revolute 5: type revolute, parent thigh_1, child knee_1, origin xyz=0.0 0.0165 -0.077 rpy=0 0 0, axis -0.0 -1.0 -0.0, limit lower=-1.57 upper=1.57 effort=100 velocity=1.0
- added joint Revolute 6: type revolute, parent knee_1, child shin_1, origin xyz=0.0 0.0 -0.031 rpy=0 0 0, axis 0.0 1.0 0.0, limit lower=-1.57 upper=1.57 effort=100 velocity=1.0
- added joint Revolute 8: type revolute, parent servo_3_1, child ankle_1, origin xyz=0.0 0.01865 -0.035 rpy=0 0 0, axis 0.0 1.0 0.0, limit lower=-1.57 upper=1.57 effort=100 velocity=1.0
- added joint Revolute 9: type revolute, parent ankle_1, child servo_4_1, origin xyz=0.01865 -0.01865 -0.04 rpy=0 0 0, axis -1.0 -0.0 0.0, limit lower=-1.57 upper=1.57 effort=100 velocity=1.0
- added joint Rigid 1: type fixed, parent base_link, child servo1_1, origin xyz=0.0 0.0 -0.002 rpy=0 0 0
- added joint Rigid 10: type fixed, parent servo_4_1, child foot_1, origin xyz=-0.01865 0.01 0.0 rpy=0 0 0
- added joint Rigid 11: type fixed, parent foot_1, child end_1, origin xyz=0.011292 0.080404 0.268287 rpy=0 0 0
- added joint Rigid 4: type fixed, parent servo_2_1, child thigh_1, origin xyz=0.0 0.01865 0.01 rpy=0 0 0
- added joint Rigid 7: type fixed, parent shin_1, child servo_3_1, origin xyz=0.0 -0.0165 -0.032 rpy=0 0 0

File: leg/Untitled_description/urdf/materials.xacro (robot description, xacro)
@@ -1,4 +1,4 @@
 <?xml version="1.0" ?>
-<robot name="Walker" xmlns:xacro="http://www.ros.org/wiki/xacro" >
+<robot name="Untitled" xmlns:xacro="http://www.ros.org/wiki/xacro" >
 <material name="silver">
   <color rgba="0.700 0.700 0.700 1.000"/>

File: trash/Walker.urdf (robot description, URDF)
Before this commit: robot Walker, 8 links, 7 joints
Links:
- removed link end_effector_1
- removed link right_ankle_1
- removed link right_foot_1
- removed link right_hip_1
- removed link right_knee_1
- removed link right_shin_1
- removed link right_thigh_1
- added link Component212_1, mass 0.7031706971853583; collision mesh filename=leg/Walker_description/meshes/Component212_1.stl scale=0.001 0.001 0.001; visual mesh filename=leg/Walker_description/meshes/Component212_1.stl scale=0.001 0.001 0.001
- added link Component215_1, mass 0.7031706971853583; collision mesh filename=leg/Walker_description/meshes/Component215_1.stl scale=0.001 0.001 0.001; visual mesh filename=leg/Walker_description/meshes/Component215_1.stl scale=0.001 0.001 0.001
- added link Component218_1, mass 0.27927069718535813; collision mesh filename=leg/Walker_description/meshes/Component218_1.stl scale=0.001 0.001 0.001; visual mesh filename=leg/Walker_description/meshes/Component218_1.stl scale=0.001 0.001 0.001
- link base_link: mass 0.027166123584619145 -> 0.27927069718535813
Joints:
- removed joint Revolute 85
- removed joint Revolute 86
- removed joint Revolute 88
- removed joint Revolute 89
- removed joint Revolute 91
- removed joint Rigid 87
- removed joint Rigid 93
- added joint Revolute 102: type revolute, parent base_link, child Component212_1, origin xyz=0.0 -0.015 -0.03 rpy=0 0 0, axis 0.0 1.0 0.0, limit lower=-1.57 upper=1.57 effort=100 velocity=1.0
- added joint Revolute 103: type revolute, parent Component212_1, child Component215_1, origin xyz=0.0 0.0 -0.08 rpy=0 0 0, axis 0.0 1.0 0.0, limit lower=0 upper=3.14 effort=100 velocity=1.0
- added joint Revolute 104: type revolute, parent Component215_1, child Component218_1, origin xyz=0.0 0.0 -0.08 rpy=0 0 0, axis 0.0 1.0 0.0, limit lower=-1.57 upper=1.57 effort=100 velocity=1.0

Commit message: r

File: Walker.urdf (robot description, URDF)
Before this commit: robot Untitled, 12 links, 11 joints
Joints:
- joint Revolute 2: limit lower=-1.57 upper=1.57 effort=100 velocity=1.0 -> (none); type revolute -> continuous
- joint Revolute 3: limit lower=-1.57 upper=1.57 effort=100 velocity=1.0 -> (none); type revolute -> continuous
- joint Revolute 5: limit lower=-1.57 upper=1.57 effort=100 velocity=1.0 -> (none); type revolute -> continuous
- joint Revolute 6: limit lower=-1.57 upper=1.57 effort=100 velocity=1.0 -> (none); type revolute -> continuous
- joint Revolute 8: limit lower=-1.57 upper=1.57 effort=100 velocity=1.0 -> (none); type revolute -> continuous
- joint Revolute 9: limit lower=-1.57 upper=1.57 effort=100 velocity=1.0 -> (none); type revolute -> continuous

Commit message: s

File: Walker.urdf (robot description, URDF)
Before this commit: robot Untitled, 12 links, 11 joints
Links:
- removed link ankle_1
- removed link end_1
- removed link hip_1
- removed link servo1_1
- removed link servo_2_1
- removed link servo_3_1
- removed link servo_4_1
- link base_link: mass 0.07564259890699374 -> 0.2792706971853582; geometry collision mesh filename=leg/Walker_description/meshes/base_link.stl scale=0.001 0.001 0.001; visual mesh filename=leg/Walker_description/meshes/base_link.stl scale=0.001 0.001 0.001
- link foot_1: mass 0.07564259890689244 -> 0.27927069718535813; geometry collision mesh filename=leg/Walker_description/meshes/foot_1.stl scale=0.001 0.001 0.001; visual mesh filename=leg/Walker_description/meshes/foot_1.stl scale=0.001 0.001 0.001
- link knee_1: mass 0.3524642857407411 -> 0.7031706971853583; geometry collision mesh filename=leg/Walker_description/meshes/knee_1.stl scale=0.001 0.001 0.001; visual mesh filename=leg/Walker_description/meshes/knee_1.stl scale=0.001 0.001 0.001
- link shin_1: mass 0.3751668513433219 -> 0.27927069718535813; geometry collision mesh filename=leg/Walker_description/meshes/shin_1.stl scale=0.001 0.001 0.001; visual mesh filename=leg/Walker_description/meshes/shin_1.stl scale=0.001 0.001 0.001
- link thigh_1: mass 0.3751668513433219 -> 0.7031706971853583; geometry collision mesh filename=leg/Walker_description/meshes/thigh_1.stl scale=0.001 0.001 0.001; visual mesh filename=leg/Walker_description/meshes/thigh_1.stl scale=0.001 0.001 0.001
Joints:
- removed joint Revolute 2
- removed joint Revolute 3
- removed joint Revolute 5
- removed joint Revolute 6
- removed joint Revolute 8
- removed joint Revolute 9
- removed joint Rigid 1
- removed joint Rigid 10
- removed joint Rigid 11
- removed joint Rigid 4
- removed joint Rigid 7
- added joint Revolute 107: type continuous, parent base_link, child thigh_1, origin xyz=0.0 0.015 -0.03 rpy=0 0 0, axis 0.0 1.0 0.0
- added joint Revolute 108: type continuous, parent thigh_1, child foot_1, origin xyz=0.0 0.0 -0.08 rpy=0 0 0, axis -0.0 1.0 -0.0
- added joint Revolute 109: type continuous, parent foot_1, child knee_1, origin xyz=0.0 0.0 -0.02 rpy=0 0 0, axis 0.0 1.0 -0.0
- added joint Revolute 110: type continuous, parent knee_1, child shin_1, origin xyz=0.0 0.0 -0.08 rpy=0 0 0, axis 0.0 1.0 -0.0

File: leg/Walker_description/urdf/materials.xacro (robot description, xacro)
@@ -1,4 +1,4 @@
 <?xml version="1.0" ?>
-<robot name="Untitled" xmlns:xacro="http://www.ros.org/wiki/xacro" >
+<robot name="Walker" xmlns:xacro="http://www.ros.org/wiki/xacro" >
 <material name="silver">
   <color rgba="0.700 0.700 0.700 1.000"/>
