Commit message: t

File: Walker.urdf (robot description, URDF)
Before this commit: robot Walker, 5 links, 4 joints
Links:
- removed link foot_1
- removed link knee_1
- removed link shin_1
- added link foot, mass 0.27927069718535813; collision mesh filename=leg/Walker_description/meshes/shin_1.stl scale=0.001 0.001 0.001; visual mesh filename=leg/Walker_description/meshes/shin_1.stl scale=0.001 0.001 0.001
- added link knee, mass 0.27927069718535813; collision mesh filename=leg/Walker_description/meshes/foot_1.stl scale=0.001 0.001 0.001; visual mesh filename=leg/Walker_description/meshes/foot_1.stl scale=0.001 0.001 0.001
- added link shin, mass 0.7031706971853583; collision mesh filename=leg/Walker_description/meshes/knee_1.stl scale=0.001 0.001 0.001; visual mesh filename=leg/Walker_description/meshes/knee_1.stl scale=0.001 0.001 0.001
Joints:
- joint Revolute 108: child foot_1 -> knee
- joint Revolute 109: child knee_1 -> shin; parent foot_1 -> knee
- joint Revolute 110: child shin_1 -> foot; parent knee_1 -> shin

Commit message: x

File: Walker.urdf (robot description, URDF)
Before this commit: robot Walker, 7 links, 6 joints
Links:
- added link hip_roll_1, mass 0.2792706971853587; collision mesh filename=leg/Walker_description/meshes/hip_roll_1.stl scale=0.001 0.001 0.001; visual mesh filename=leg/Walker_description/meshes/hip_roll_1.stl scale=0.001 0.001 0.001
- link ankle_1: mass 0.2763113169056768 -> 0.27927069718535824
- link ankle_roll_1: mass 0.2733519366259955 -> 0.2792706971853587
- link base_link: mass 0.2792706971853582 -> 0.28093534859267927
Joints:
- removed joint Revolute 112
- removed joint Rigid 113
- removed joint ankle
- removed joint hip
- removed joint knee_1
- removed joint knee_2
- added joint Rigid 120: type fixed, parent ankle_roll_1, child foot_1, origin xyz=-0.015 0.0 -0.03 rpy=0 0 0
- added joint ankle_pitch: type continuous, parent shin_1, child ankle_1, origin xyz=0.0 0.0 -0.08 rpy=0 0 0, axis 0.0 1.0 -0.0
- added joint ankle_roll: type continuous, parent ankle_1, child ankle_roll_1, origin xyz=0.015 -0.015 -0.02 rpy=0 0 0, axis 1.0 -0.0 0.0
- added joint hip_pitch: type continuous, parent hip_roll_1, child thigh_1, origin xyz=-0.015 0.015 -0.02 rpy=0 0 0, axis -0.0 -1.0 0.0
- added joint hip_roll: type continuous, parent base_link, child hip_roll_1, origin xyz=0.015 0.0 -0.03 rpy=0 0 0, axis 1.0 0.0 0.0
- added joint knee_pitch1: type continuous, parent thigh_1, child knee_1, origin xyz=0.0 0.0 -0.08 rpy=0 0 0, axis -0.0 1.0 -0.0
- added joint knee_pitch2: type continuous, parent knee_1, child shin_1, origin xyz=0.0 0.0 -0.02 rpy=0 0 0, axis 0.0 1.0 -0.0

File: leg/Walker_description/urdf/Walker.xacro (robot description, xacro)
@@ -6,7 +6,7 @@
 <link name="base_link">
   <inertial>
-    <origin xyz="-1.8714321332029245e-15 -1.997259480472705e-18 -0.020000000000000004" rpy="0 0 0"/>
-    <mass value="0.2792706971853582"/>
-    <inertia ixx="5.8e-05" iyy="5.9e-05" izz="4.2e-05" ixy="-0.0" iyz="-0.0" ixz="-0.0"/>
+    <origin xyz="0.0 0.0 -0.019940746103482097" rpy="0 0 0"/>
+    <mass value="0.28093534859267927"/>
+    <inertia ixx="5.9e-05" iyy="5.9e-05" izz="4.2e-05" ixy="0.0" iyz="0.0" ixz="0.0"/>
   </inertial>
   <visual>
@@ -24,12 +24,32 @@
   </collision>
 </link>
+<link name="hip_roll_1">
+  <inertial>
+    <origin xyz="-0.015000000000000097 8.898885287580091e-16 -0.009999999999998191" rpy="0 0 0"/>
+    <mass value="0.2792706971853587"/>
+    <inertia ixx="5.8e-05" iyy="5.8e-05" izz="4.2e-05" ixy="0.0" iyz="-0.0" ixz="0.0"/>
+  </inertial>
+  <visual>
+    <origin xyz="-0.015 -0.0 0.03" rpy="0 0 0"/>
+    <geometry>
+      <mesh filename="package://Walker_description/meshes/hip_roll_1.stl" scale="0.001 0.001 0.001"/>
+    </geometry>
+    <material name="silver"/>
+  </visual>
+  <collision>
+    <origin xyz="-0.015 -0.0 0.03" rpy="0 0 0"/>
+    <geometry>
+      <mesh filename="package://Walker_description/meshes/hip_roll_1.stl" scale="0.001 0.001 0.001"/>
+    </geometry>
+  </collision>
+</link>
 <link name="thigh_1">
   <inertial>
-    <origin xyz="-3.049337275221765e-16 -0.01499999999999996 -0.04000000000000009" rpy="0 0 0"/>
+    <origin xyz="-3.675018476364042e-16 -0.015000000000000213 -0.040000000000000216" rpy="0 0 0"/>
     <mass value="0.7031706971853584"/>
     <inertia ixx="0.000636" iyy="0.000636" izz="0.000106" ixy="-0.0" iyz="-0.0" ixz="0.0"/>
   </inertial>
   <visual>
-    <origin xyz="-0.0 -0.015 0.03" rpy="0 0 0"/>
+    <origin xyz="0.0 -0.015 0.05" rpy="0 0 0"/>
     <geometry>
       <mesh filename="package://Walker_description/meshes/thigh_1.stl" scale="0.001 0.001 0.001"/>
@@ -38,5 +58,5 @@
   </visual>
   <collision>
-    <origin xyz="-0.0 -0.015 0.03" rpy="0 0 0"/>
+    <origin xyz="0.0 -0.015 0.05" rpy="0 0 0"/>
     <geometry>
       <mesh filename="package://Walker_description/meshes/thigh_1.stl" scale="0.001 0.001 0.001"/>
@@ -46,10 +66,10 @@
 <link name="knee_1">
   <inertial>
-    <origin xyz="-1.711783204225683e-15 -0.015000000000000025 -0.009999999999999662" rpy="0 0 0"/>
+    <origin xyz="-1.7593300251577167e-15 -0.01499999999999996 -0.009999999999999898" rpy="0 0 0"/>
     <mass value="0.27927069718535813"/>
-    <inertia ixx="5.8e-05" iyy="5.9e-05" izz="4.2e-05" ixy="-0.0" iyz="0.0" ixz="-0.0"/>
-  </inertial>
-  <visual>
-    <origin xyz="-0.0 -0.015 0.11" rpy="0 0 0"/>
+    <inertia ixx="5.8e-05" iyy="5.9e-05" izz="4.2e-05" ixy="0.0" iyz="-0.0" ixz="-0.0"/>
+  </inertial>
+  <visual>
+    <origin xyz="-0.0 -0.015 0.13" rpy="0 0 0"/>
     <geometry>
       <mesh filename="package://Walker_description/meshes/knee_1.stl" scale="0.001 0.001 0.001"/>
@@ -58,5 +78,5 @@
   </visual>
   <collision>
-    <origin xyz="-0.0 -0.015 0.11" rpy="0 0 0"/>
+    <origin xyz="-0.0 -0.015 0.13" rpy="0 0 0"/>
     <geometry>
       <mesh filename="package://Walker_description/meshes/knee_1.stl" scale="0.001 0.001 0.001"/>
@@ -66,10 +86,10 @@
 <link name="shin_1">
   <inertial>
-    <origin xyz="5.248353996103225e-09 -0.014999999999999979 -0.03999998244649294" rpy="0 0 0"/>
+    <origin xyz="5.248353906337566e-09 -0.014999999999999809 -0.03999998244649275" rpy="0 0 0"/>
     <mass value="0.7031704499676481"/>
-    <inertia ixx="0.000636" iyy="0.000636" izz="0.000106" ixy="-0.0" iyz="-0.0" ixz="0.0"/>
-  </inertial>
-  <visual>
-    <origin xyz="-0.0 -0.015 0.13" rpy="0 0 0"/>
+    <inertia ixx="0.000636" iyy="0.000636" izz="0.000106" ixy="0.0" iyz="-0.0" ixz="0.0"/>
+  </inertial>
+  <visual>
+    <origin xyz="-0.0 -0.015 0.15" rpy="0 0 0"/>
     <geometry>
       <mesh filename="package://Walker_description/meshes/shin_1.stl" scale="0.001 0.001 0.001"/>
@@ -78,5 +98,5 @@
   </visual>
   <collision>
-    <origin xyz="-0.0 -0.015 0.13" rpy="0 0 0"/>
+    <origin xyz="-0.0 -0.015 0.15" rpy="0 0 0"/>
     <geometry>
       <mesh filename="package://Walker_description/meshes/shin_1.stl" scale="0.001 0.001 0.001"/>
@@ -86,10 +106,10 @@
 <link name="ankle_1">
   <inertial>
-    <origin xyz="-6.614160307778296e-16 -0.015000000000000046 -0.009892896884822783" rpy="0 0 0"/>
-    <mass value="0.2763113169056768"/>
+    <origin xyz="-7.240003152659723e-16 -0.015000000000000237 -0.009999999999997067" rpy="0 0 0"/>
+    <mass value="0.27927069718535824"/>
     <inertia ixx="5.8e-05" iyy="5.8e-05" izz="4.2e-05" ixy="-0.0" iyz="-0.0" ixz="0.0"/>
   </inertial>
   <visual>
-    <origin xyz="-0.0 -0.015 0.21" rpy="0 0 0"/>
+    <origin xyz="-0.0 -0.015 0.23" rpy="0 0 0"/>
     <geometry>
       <mesh filename="package://Walker_description/meshes/ankle_1.stl" scale="0.001 0.001 0.001"/>
@@ -98,5 +118,5 @@
   </visual>
   <collision>
-    <origin xyz="-0.0 -0.015 0.21" rpy="0 0 0"/>
+    <origin xyz="-0.0 -0.015 0.23" rpy="0 0 0"/>
     <geometry>
       <mesh filename="package://Walker_description/meshes/ankle_1.stl" scale="0.001 0.001 0.001"/>
@@ -106,10 +126,10 @@
 <link name="ankle_roll_1">
   <inertial>
-    <origin xyz="-0.01499999999999974 4.2700459907529125e-15 -0.009999999999990933" rpy="0 0 0"/>
-    <mass value="0.2733519366259955"/>
-    <inertia ixx="5.8e-05" iyy="5.8e-05" izz="4.2e-05" ixy="0.0" iyz="-0.0" ixz="0.0"/>
-  </inertial>
-  <visual>
-    <origin xyz="-0.015 0.0 0.23" rpy="0 0 0"/>
+    <origin xyz="-0.014999999999999404 6.39785483460577e-16 -0.009999999999997178" rpy="0 0 0"/>
+    <mass value="0.2792706971853587"/>
+    <inertia ixx="5.8e-05" iyy="5.8e-05" izz="4.2e-05" ixy="0.0" iyz="-0.0" ixz="-0.0"/>
+  </inertial>
+  <visual>
+    <origin xyz="-0.015 0.0 0.25" rpy="0 0 0"/>
     <geometry>
       <mesh filename="package://Walker_description/meshes/ankle_roll_1.stl" scale="0.001 0.001 0.001"/>
@@ -118,5 +138,5 @@
   </visual>
   <collision>
-    <origin xyz="-0.015 0.0 0.23" rpy="0 0 0"/>
+    <origin xyz="-0.015 0.0 0.25" rpy="0 0 0"/>
     <geometry>
       <mesh filename="package://Walker_description/meshes/ankle_roll_1.stl" scale="0.001 0.001 0.001"/>
@@ -126,10 +146,10 @@
 <link name="foot_1">
   <inertial>
-    <origin xyz="2.0932740912099903e-16 -1.4558288635419128e-16 -0.004999999999999838" rpy="0 0 0"/>
+    <origin xyz="6.245004505575571e-16 -2.76128590171539e-16 -0.004999999999999394" rpy="0 0 0"/>
     <mass value="0.5024"/>
-    <inertia ixx="0.000272" iyy="0.000272" izz="0.000536" ixy="0.0" iyz="0.0" ixz="0.0"/>
-  </inertial>
-  <visual>
-    <origin xyz="-0.0 0.0 0.26" rpy="0 0 0"/>
+    <inertia ixx="0.000272" iyy="0.000272" izz="0.000536" ixy="0.0" iyz="-0.0" ixz="-0.0"/>
+  </inertial>
+  <visual>
+    <origin xyz="-0.0 0.0 0.28" rpy="0 0 0"/>
     <geometry>
       <mesh filename="package://Walker_description/meshes/foot_1.stl" scale="0.001 0.001 0.001"/>
@@ -138,5 +158,5 @@
   </visual>
   <collision>
-    <origin xyz="-0.0 0.0 0.26" rpy="0 0 0"/>
+    <origin xyz="-0.0 0.0 0.28" rpy="0 0 0"/>
     <geometry>
       <mesh filename="package://Walker_description/meshes/foot_1.stl" scale="0.001 0.001 0.001"/>
@@ -144,11 +164,17 @@
   </collision>
 </link>
-<joint name="hip" type="continuous">
-  <origin xyz="0.0 0.015 -0.03" rpy="0 0 0"/>
+<joint name="hip_roll" type="continuous">
+  <origin xyz="0.015 0.0 -0.03" rpy="0 0 0"/>
   <parent link="base_link"/>
+  <child link="hip_roll_1"/>
+  <axis xyz="1.0 0.0 0.0"/>
+</joint>
+<joint name="hip_pitch" type="continuous">
+  <origin xyz="-0.015 0.015 -0.02" rpy="0 0 0"/>
+  <parent link="hip_roll_1"/>
   <child link="thigh_1"/>
-  <axis xyz="0.0 1.0 0.0"/>
-</joint>
-<joint name="knee_1" type="continuous">
+  <axis xyz="-0.0 -1.0 0.0"/>
+</joint>
+<joint name="knee_pitch1" type="continuous">
   <origin xyz="0.0 0.0 -0.08" rpy="0 0 0"/>
   <parent link="thigh_1"/>
@@ -156,5 +182,5 @@
   <axis xyz="-0.0 1.0 -0.0"/>
 </joint>
-<joint name="knee_2" type="continuous">
+<joint name="knee_pitch2" type="continuous">
   <origin xyz="0.0 0.0 -0.02" rpy="0 0 0"/>
   <parent link="knee_1"/>
@@ -162,5 +188,5 @@
   <axis xyz="0.0 1.0 -0.0"/>
 </joint>
-<joint name="ankle" type="continuous">
+<joint name="ankle_pitch" type="continuous">
   <origin xyz="0.0 0.0 -0.08" rpy="0 0 0"/>
   <parent link="shin_1"/>
@@ -168,5 +194,5 @@
   <axis xyz="0.0 1.0 -0.0"/>
 </joint>
-<joint name="Revolute 112" type="continuous">
+<joint name="ankle_roll" type="continuous">
   <origin xyz="0.015 -0.015 -0.02" rpy="0 0 0"/>
   <parent link="ankle_1"/>
@@ -174,5 +200,5 @@
   <axis xyz="1.0 -0.0 0.0"/>
 </joint>
-<joint name="Rigid 113" type="fixed">
+<joint name="Rigid 120" type="fixed">
   <origin xyz="-0.015 0.0 -0.03" rpy="0 0 0"/>
   <parent link="ankle_roll_1"/>

Commit message: a

File: Walker.urdf (robot description, URDF)
Before this commit: robot Walker, 8 links, 7 joints
Links:
- removed link ankle_roll_1
- removed link hip_roll_1
- added link end_1, mass 0.23876488296307571; collision mesh filename=walker/Walker_description/meshes/end_1.stl scale=0.001 0.001 0.001; visual mesh filename=walker/Walker_description/meshes/end_1.stl scale=0.001 0.001 0.001
- added link hip_1, mass 0.1612694354483246; collision mesh filename=walker/Walker_description/meshes/hip_1.stl scale=0.001 0.001 0.001; visual mesh filename=walker/Walker_description/meshes/hip_1.stl scale=0.001 0.001 0.001
- link ankle_1: mass 0.27927069718535824 -> 0.16126943544832473; geometry collision mesh filename=walker/Walker_description/meshes/ankle_1.stl scale=0.001 0.001 0.001; visual mesh filename=walker/Walker_description/meshes/ankle_1.stl scale=0.001 0.001 0.001
- link base_link: mass 0.28093534859267927 -> 0.3640061961261434; geometry collision mesh filename=walker/Walker_description/meshes/base_link.stl scale=0.001 0.001 0.001; visual mesh filename=walker/Walker_description/meshes/base_link.stl scale=0.001 0.001 0.001
- link foot_1: mass 0.5024 -> 0.3639507075296119; geometry collision mesh filename=walker/Walker_description/meshes/foot_1.stl scale=0.001 0.001 0.001; visual mesh filename=walker/Walker_description/meshes/foot_1.stl scale=0.001 0.001 0.001
- link knee_1: mass 0.27927069718535813 -> 0.3524642857407411; geometry collision mesh filename=walker/Walker_description/meshes/knee_1.stl scale=0.001 0.001 0.001; visual mesh filename=walker/Walker_description/meshes/knee_1.stl scale=0.001 0.001 0.001
- link shin_1: mass 0.7031704499676481 -> 0.663530448562467; geometry collision mesh filename=walker/Walker_description/meshes/shin_1.stl scale=0.001 0.001 0.001; visual mesh filename=walker/Walker_description/meshes/shin_1.stl scale=0.001 0.001 0.001
- link thigh_1: mass 0.7031706971853584 -> 0.6635304485624715; geometry collision mesh filename=walker/Walker_description/meshes/thigh_1.stl scale=0.001 0.001 0.001; visual mesh filename=walker/Walker_description/meshes/thigh_1.stl scale=0.001 0.001 0.001
Joints:
- removed joint Rigid 120
- removed joint ankle_pitch
- removed joint ankle_roll
- removed joint hip_pitch
- removed joint hip_roll
- removed joint knee_pitch1
- removed joint knee_pitch2
- added joint Revolute 31: type continuous, parent base_link, child hip_1, origin xyz=0.01865 0.0 -0.037 rpy=0 0 0, axis 1.0 -0.0 0.0, limit lower=-1.57 upper=1.57 effort=100 velocity=1.0
- added joint Revolute 32: type continuous, parent hip_1, child thigh_1, origin xyz=-0.01865 0.01865 -0.04 rpy=0 0 0, axis -0.0 1.0 -0.0, limit lower=-1.57 upper=0.78 effort=100 velocity=1.0
- added joint Revolute 33: type continuous, parent thigh_1, child knee_1, origin xyz=0.0 -0.00215 -0.067 rpy=0 0 0, axis -0.0 -1.0 0.0, limit lower=-3.14 upper=3.14 effort=100 velocity=1.0
- added joint Revolute 34: type continuous, parent knee_1, child shin_1, origin xyz=0.0 0.0 -0.031 rpy=0 0 0, axis 0.0 1.0 -0.0, limit lower=0 upper=1.57 effort=100 velocity=1.0
- added joint Revolute 35: type continuous, parent shin_1, child ankle_1, origin xyz=0.0 0.00215 -0.067 rpy=0 0 0, axis -0.0 1.0 0.0
- added joint Revolute 36: type continuous, parent ankle_1, child foot_1, origin xyz=0.01865 -0.01865 -0.04 rpy=0 0 0, axis 1.0 -0.0 0.0
- added joint Rigid 37: type fixed, parent foot_1, child end_1, origin xyz=-0.01865 0.0 -0.014 rpy=0 0 0

Commit message: e

File: Walker.urdf (robot description, URDF)
Before this commit: robot Walker, 8 links, 7 joints
Joints:
- joint Revolute 31: limit lower=-1.57 upper=1.57 effort=100 velocity=1.0 -> (none)
- joint Revolute 32: limit lower=-1.57 upper=0.78 effort=100 velocity=1.0 -> (none)
- joint Revolute 33: limit lower=-3.14 upper=3.14 effort=100 velocity=1.0 -> (none)
- joint Revolute 34: limit lower=0 upper=1.57 effort=100 velocity=1.0 -> (none)
