Commit message: c

File: Walker2.urdf (robot description, URDF)
Before this commit: robot Walker, 15 links, 14 joints
Joints:
- joint Revolute 32: limit (none) -> lower=-1.57 upper=1.57 effort=100 velocity=1.0; type continuous -> revolute
- joint Revolute 33: limit (none) -> lower=-3.14 upper=3.14 effort=100 velocity=1.0; type continuous -> revolute
- joint Revolute 34: limit (none) -> lower=0 upper=1.57 effort=100 velocity=1.0; type continuous -> revolute
- joint Revolute 35: limit (none) -> lower=-1.57 upper=1.57 effort=100 velocity=1.0; type continuous -> revolute
- joint Revolute 36: limit (none) -> lower=-1.57 upper=1.57 effort=100 velocity=1.0; type continuous -> revolute
- joint Revolute 39: limit (none) -> lower=-1.57 upper=1.57 effort=100 velocity=1.0; type continuous -> revolute
- joint Revolute 40: limit (none) -> lower=-3.14 upper=3.14 effort=100 velocity=1.0; type continuous -> revolute
- joint Revolute 41: limit (none) -> lower=-1.57 upper=0 effort=100 velocity=1.0; type continuous -> revolute
- joint Revolute 42: limit (none) -> lower=-1.57 upper=1.57 effort=100 velocity=1.0; type continuous -> revolute
- joint Revolute 43: limit (none) -> lower=-1.57 upper=1.57 effort=100 velocity=1.0; type continuous -> revolute
- joint Revolute 46: limit (none) -> lower=-1.57 upper=1.57 effort=100 velocity=1.0; type continuous -> revolute
- joint Revolute 47: limit (none) -> lower=-1.57 upper=1.57 effort=100 velocity=1.0; type continuous -> revolute

Commit message: l

File: Walker2.urdf (robot description, URDF)
Before this commit: robot Walker, 15 links, 14 joints
Links:
- link base_link: mass 1.3880717876460764 -> 0.4
